File: hardware/cx-jig-kicad/vt610ex-sc3a-clock-gen-adapter.kicad_pcb (KiCad board)
At the start: 2 copper layers, 20.2 x 12 mm, 10 parts, among them J11 Conn_01x01_Pin, J12 Conn_01x01_Pin, J21 Conn_01x01_Pin, J22 Conn_01x01_Pin, J30 Conn_Coaxial

Commit message: Remove obsolete KiCad project files for the clock generator main board, including DRC, ERC, DRU, PCB, schematic, and project configuration files. Updated the CX Jig project files with new author and company details, modified component properties, and adjusted net definitions for improved clarity and organization.
Parts:
- J1: renamed from J30; footprint Connector_Coaxial:SMA_Samtec_SMA-J-P-X-ST-EM1_EdgeMount -> Connector_Coaxial:SMA_Samtec_SMA-J-P-H-ST-EM1_EdgeMount
- moved J1 0.26 mm to (143.2, 81.0), turned to 0 degrees
- renumbered J11 to J2, J12 to J3, J21 to J4, J22 to J5
Connections:
- net /vcc_33 renamed /V_{cc}_3V3
- net /xt1 renamed /XT1
- net /xt2 renamed /XT2
