File: kicad/main-board.kicad_sch (KiCad schematic)
At the start: 15 parts, among them J1 Conn_01x03_Pin, J2 Conn_01x03_Pin, J3 Headswitch_SMA, J8 Conn_Coaxial, U1 Pico

Commit message: Remove obsolete KiCad project files for the clock generator main board, including DRC, ERC, DRU, PCB, schematic, and project configuration files. Updated the CX Jig project files with new author and company details, modified component properties, and adjusted net definitions for improved clarity and organization.
Parts:
- renumbered D2 to D1, D1 to D2, J3 to J1, J8 to J2, J2 to J3, J1 to J4, U3 to U2, U2 to U3
Connections:
- net Head_SW_In: now reaches D1.2 (A), J1.1, J2.1 (In)
Other:
- company: ${proj-author} -> ${proj-company}
- title: ${proj-title} -> Main Board
